File: Schematic/CG1111A_MBOT/CG1111A_MBOT.kicad_sch (KiCad schematic)
At the start: 20 parts

Commit message: feat: lab2
Parts:
- R?: value R -> 1.5k
- R?: value R -> 800
- R?: value R -> 5.6k
Other:
- note added: "Port 3 S1 - A2 S2 - A3"
- note added: "Port 4 S1 - A0 S2 - A1"
Changed lines of the file:
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@@
     (stroke (width 0) (type default) (color 0 0 0 0))
+  )
+  (text "Port 3\n\nS1 - A2\nS2 - A3\n" (at 17.78 138.43 0)
+    (effects (font (size 1.27 1.27)) (justify left bottom))
   )
   (text "LDR " (at 177.8 59.69 0)
@@
     (effects (font (size 4 4) bold) (justify left bottom))
   )
+  (text "Port 4\n\nS1 - A0\nS2 - A1\n" (at 19.05 54.61 0)
+    (effects (font (size 1.27 1.27)) (justify left bottom))
+  )
   (text "Breadboard 2" (at 22.86 100.33 0)
     (effects (font (size 4 4) bold) (justify left bottom))
@@
       (effects (font (size 1.27 1.27)) (justify left))
     )
-    (property "Value" "R" (id 1) (at 162.56 41.9099 0)
+    (property "Value" "1.5k" (id 1) (at 162.56 41.9099 0)
       (effects (font (size 1.27 1.27)) (justify left))
     )
@@
       (effects (font (size 1.27 1.27)) (justify left))
     )
-    (property "Value" "R" (id 1) (at 143.51 41.9099 0)
+    (property "Value" "800" (id 1) (at 143.51 41.9099 0)
       (effects (font (size 1.27 1.27)) (justify left))
     )
@@
       (effects (font (size 1.27 1.27)) (justify left))
     )
-    (property "Value" "R" (id 1) (at 152.4 41.9099 0)
+    (property "Value" "5.6k" (id 1) (at 152.4 41.9099 0)
       (effects (font (size 1.27 1.27)) (justify left))
     )
@@
     )
     (path "/02879672-67cc-4352-922e-f581dd7be20d"
-      (reference "R?") (unit 1) (value "R") (footprint "")
+      (reference "R?") (unit 1) (value "1.5k") (footprint "")
     )
     (path "/35be63c5-5965-410d-8398-2dfe7a3c4cf8"
@@
     )
     (path "/3ccae707-0b86-4d62-9117-edc18f684ca7"
-      (reference "R?") (unit 1) (value "R") (footprint "")
+      (reference "R?") (unit 1) (value "800") (footprint "")
     )
     (path "/449c78e2-aa5d-4c4a-ac04-a248a680b46c"
@@
     )
     (path "/5d96db6c-48ce-4ef2-9744-50cd5f00fc83"
-      (reference "R?") (unit 1) (value "R") (footprint "")
+      (reference "R?") (unit 1) (value "5.6k") (footprint "")
     )
     (path "/96bb075a-11af-4fde-b09d-b2d8c92aea7d"

Commit message: feat: temp
Parts:
- R?: value R -> 8k
Changed lines of the file:
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@@
       (effects (font (size 1.27 1.27)) (justify left))
     )
-    (property "Value" "R" (id 1) (at 153.67 133.3499 0)
+    (property "Value" "8k" (id 1) (at 153.67 133.3499 0)
       (effects (font (size 1.27 1.27)) (justify left))
     )
@@
     )
     (path "/35be63c5-5965-410d-8398-2dfe7a3c4cf8"
-      (reference "R?") (unit 1) (value "R") (footprint "")
+      (reference "R?") (unit 1) (value "8k") (footprint "")
     )
     (path "/3ccae707-0b86-4d62-9117-edc18f684ca7"
