File: Schematic/CG1111A_MBOT/CG1111A_MBOT.kicad_sch (KiCad schematic)
At the start: 20 parts

Commit message: chore: cleanup code - MOCK RUN READY
Parts:
- R1: renamed from R?; value R -> 150
- gave numbers to parts that had none: 17
Other:
- note added: "IR LED in Practice : ranges from 0.8V (when high) to 1.2V (when low)"
- note added: "Ideal 5V / 150ohm = 33mA"
- note added: "Minimum Resistor value: 5V/8mA = 625ohm Brightness -> Current -> LED Red Green Blue"
- note removed: "Resistor value: 5V/8mA = 625ohm Brightness -> Current -> LED Red Green Blue"
- moved on the sheet: Q1, R4
